File: PCB/flsh/flsh.kicad_pcb (KiCad board)
At the start: 2 copper layers, 40 x 40 mm, 21 parts, among them M1 IAUCN04S7L028ATMA1, U1 LM3478MM

Commit message: various pcb improvements and musings
Parts:
- moved TP1 6.40 mm to (134.5, 48.5)
- moved TP3 5.40 mm to (136.0, 55.0)
- moved Rfadj1 1.71 mm to (141.7, 54.0), turned to -110 degrees
- moved CComp2 1.00 mm to (146.5, 55.5), turned to -20 degrees
- moved Cbyp1 1.00 mm to (139.5, 46.0)
Routing:
- net Net-(D1-A): track 31.6 -> 25.5 mm
- net GND: track 18.1 -> 13.8 mm, vias 2 -> 18
- net Net-(M1-S): track 12.1 -> 10.1 mm
- net /DR: track 12.7 -> 11.7 mm
- net IOUT: track 46.8 -> 46.2 mm
- net Net-(U1-FB): track 7.13 -> 6.58 mm
- net Net-(U1-FA/SD): track 4.51 -> 3.97 mm
- net /COMP: track 12.1 -> 12.2 mm, vias 4 -> 3

Commit message: lwk redid the whole pcb
Parts:
- removed CComp1: 150nF 16V, easyeda2kicad:C0805
- removed CComp2: 8.2nF 50V X7R, easyeda2kicad:C0805
- removed CFILT1: 10pF, easyeda2kicad:C0805
- removed CIN1, CIN2: UUD1E471MNL1GS, easyeda2kicad:CAP-SMD_BD10.0-L10.3-W10.3-LS11.0-FD
- removed Cbyp1: 100nF 25V X7R 0805, easyeda2kicad:C0805
- removed Cout1: EEHZA1H101P, easyeda2kicad:CAP-SMD_BD10.0-L10.3-W10.3-FD
- removed M1: IAUCN04S7L028ATMA1, easyeda2kicad:TDSON-8_L6.0-W5.0-P1.27-LS6.2-BL_1
- removed RCOMP1: 2.21k, easyeda2kicad:R0805
- removed RFB1: 976Ω, easyeda2kicad:R0805
- removed RFB2: 12kΩ, easyeda2kicad:R0805
- removed RFILT1: 100Ω, easyeda2kicad:R0805
- removed Rfadj1: 105kΩ, easyeda2kicad:R0805
- removed Rsense1: 3mΩ 1W sense, easyeda2kicad:RES-SMD_L6.4-W3.2-A
- removed U1: LM3478MM, easyeda2kicad:VSSOP-8_L3.0-W3.0-P0.65-LS5.0-BL
- added C1: 47uF 35V, easyeda2kicad:C2220, F.Cu at (137.7, 39.8)
- added C2: 100uF 63V, easyeda2kicad:CAP-SMD_BD10.0-L10.3-W10.3-FD, F.Cu at (158.5, 55.5)
- added C3: 1uF, easyeda2kicad:C1206, F.Cu at (133.7, 48.8)
- added C4: 1uF, easyeda2kicad:C1206, F.Cu at (161.6, 42.1)
- added RS1: JER2512F2R220, easyeda2kicad:RES-SMD_L6.4-W3.2-R2512, F.Cu at (146.0, 62.8)
- added TP5_EN1: TestPoint, TestPoint:TestPoint_Pad_D4.0mm, F.Cu at (154.0, 63.8)
- added U2: XL6006E1, easyeda2kicad:TO-263-5_L10.2-W9.9-P1.70-LS14.4-TL, F.Cu at (141.9, 54.4)
- D1: value SS24FL -> SS38_C64999; footprint easyeda2kicad:SOD-123FL_L2.8-W1.8-LS3.6-RD -> easyeda2kicad:SMA_L4.4-W2.8-LS5.4-RD
- L1: value XAL1010-562MED -> YSPI1365-470M; footprint easyeda2kicad:IND-SMD_L11.3-W10.0_XAL1010-332ME -> easyeda2kicad:IND-SMD_L13.8-W12.6_H6.5
- moved L1 21.9 mm to (149.0, 40.9), turned to -90 degrees
- moved TP1 13.8 mm to (138.2, 61.8)
- moved D1 10.5 mm to (157.2, 43.5), turned to -90 degrees
- moved TP3 8.46 mm to (138.8, 47.0)
- moved TP2 0.32 mm to (165.7, 46.5)
Connections:
- net IOUT renamed VOUT
Routing:
- net VOUT: track 46.2 -> 18.8 mm, vias 6 -> 0
- net Net-(U2-EN): track 0.00 -> 22.0 mm, vias 0 -> 2
- net VIN: track 0.00 -> 15.0 mm
- net Net-(D1-A): track 25.5 -> 10.7 mm
- net GND: track 13.8 -> 0.00 mm, vias 18 -> 15
- net Net-(U2-FB): track 0.00 -> 12.9 mm, vias 0 -> 2
- net /COMP: track 12.2 -> 0.00 mm, vias 3 -> 0
- net /DR: track 11.7 -> 0.00 mm
- net /ISEN: track 11.4 -> 0.00 mm
- net Net-(M1-S): track 10.1 -> 0.00 mm
- net Net-(U1-FB): track 6.58 -> 0.00 mm
- net Net-(U1-FA/SD): track 3.97 -> 0.00 mm
- net Net-(CComp1-Pad1): track 2.50 -> 0.00 mm
- added copper zone on F.Cu, net Net-(D1-A)
Other:
- board text added: "VOUT"
- board text removed: "IOUT"

Commit message: tiny changes
Parts:
- moved C1 1.65 mm to (139.2, 39.3), turned to -90 degrees
Routing:
- net VIN: track 15.0 -> 12.6 mm
Changed lines of the file:
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@@
 	(footprint "easyeda2kicad:C2220"
 		(layer "F.Cu")
-		(at 137.675664 39.824336 -135)
+		(at 139.25 39.330001 -90)
 		(property "Reference" "C1"
-			(at -0.898234 -3.929781 45)
+			(at -0.898234 -3.92978 90)
 			(layer "F.SilkS")
 			(effects
@@
 		)
 		(property "Value" "47uF 35V"
-			(at 0 4 45)
+			(at 0 4 90)
 			(layer "F.Fab")
 			(effects
@@
 		)
 		(property "Datasheet" "https://www.lcsc.com/datasheet/C49297048.pdf"
-			(at 0 0 45)
+			(at 0 0 90)
 			(layer "F.Fab")
 			(hide yes)
@@
 		)
 		(property "Description" ""
-			(at 0 0 45)
+			(at 0 0 90)
 			(layer "F.Fab")
 			(hide yes)
@@
 		)
 		(property "LCSC Part" "C49297048"
-			(at 0 0 45)
+			(at 0 0 90)
 			(layer "F.Fab")
 			(hide yes)
@@
 		)
 		(property "Manufacturer" "TDK"
-			(at 0 0 225)
+			(at 0 0 270)
 			(unlocked yes)
 			(layer "F.Fab")
@@
 		)
 		(property "MPN" "CKG57NX7R1H476MT009W"
-			(at 0 0 225)
+			(at 0 0 270)
 			(unlocked yes)
 			(layer "F.Fab")
@@
 		(duplicate_pad_numbers_are_jumpers no)
 		(fp_line
+			(start -1.649999 2.929999)
+			(end -3.660001 2.929999)
+			(stroke
+				(width 0.15)
+				(type solid)
+			)
+			(layer "F.SilkS")
+		)
+		(fp_line
+			(start 1.65 2.929999)
+			(end 3.66 2.93)
+			(stroke
+				(width 0.15)
+				(type solid)
+			)
+			(layer "F.SilkS")
+		)
+		(fp_line
+			(start -3.809999 2.78)
+			(end -3.81 -2.78)
+			(stroke
+				(width 0.15)
+				(type solid)
+			)
+			(layer "F.SilkS")
+		)
+		(fp_line
 			(start 3.81 2.78)
 			(end 3.809999 -2.78)
@@
 		)
 		(fp_line
-			(start 1.65 2.929999)
-			(end 3.66 2.93)
-			(stroke
-				(width 0.15)
-				(type solid)
-			)
-			(layer "F.SilkS")
-		)
-		(fp_line
-			(start -1.65 2.929999)
-			(end -3.66 2.929999)
-			(stroke
-				(width 0.15)
-				(type solid)
-			)
-			(layer "F.SilkS")
-		)
-		(fp_line
-			(start 3.66 -2.929999)
-			(end 1.65 -2.929999)
-			(stroke
-				(width 0.15)
-				(type solid)
-			)
-			(layer "F.SilkS")
-		)
-		(fp_line
-			(start -3.809999 2.78)
-			(end -3.81 -2.78)
+			(start 3.660001 -2.929999)
+			(end 1.649999 -2.929999)
 			(stroke
 				(width 0.15)
@@
 			(start -3.66 -2.93)
 			(end -1.65 -2.929999)
+			(stroke
+				(width 0.15)
+				(type solid)
+			)
+			(layer "F.SilkS")
+		)
+		(fp_arc
+			(start -3.660001 2.929999)
+			(mid -3.766066 2.886066)
+			(end -3.809999 2.78)
 			(stroke
 				(width 0.15)
@@
 		)
 		(fp_arc
-			(start 3.66 -2.929999)
-			(mid 3.766066 -2.886066)
-			(end 3.809999 -2.78)
-			(stroke
-				(width 0.15)
-				(type solid)
-			)
-			(layer "F.SilkS")
-		)
-		(fp_arc
-			(start -3.66 2.929999)
-			(mid -3.766066 2.886066)
-			(end -3.809999 2.78)
-			(stroke
-				(width 0.15)
-				(type solid)
-			)
-			(layer "F.SilkS")
-		)
-		(fp_arc
 			(start -3.81 -2.78)
 			(mid -3.766066 -2.886066)
@@
 			(layer "F.SilkS")
 		)
+		(fp_arc
+			(start 3.660001 -2.929999)
+			(mid 3.766066 -2.886066)
+			(end 3.809999 -2.78)
+			(stroke
+				(width 0.15)
+				(type solid)
+			)
+			(layer "F.SilkS")
+		)
 		(fp_circle
-			(center -2.850001 2.5)
+			(center -2.85 2.5)
 			(end -2.82 2.5)
 			(stroke
@@
 		)
 		(fp_line
+			(start -2.85 2.5)
+			(end -2.85 -2.499999)
+			(stroke
+				(width 0.05)
+				(type solid)
+			)
+			(layer "F.CrtYd")
+		)
+		(fp_line
 			(start 2.85 2.499999)
-			(end -2.850001 2.5)
+			(end -2.85 2.5)
 			(stroke
 				(width 0.05)
@@
 		)
 		(fp_line
-			(start 2.850001 -2.5)
+			(start -2.85 -2.499999)
+			(end 2.85 -2.5)
+			(stroke
+				(width 0.05)
+				(type solid)
+			)
+			(layer "F.CrtYd")
+		)
+		(fp_line
+			(start 2.85 -2.5)
 			(end 2.85 2.499999)
 			(stroke
@@
 			(layer "F.CrtYd")
 		)
-		(fp_line
-			(start -2.850001 2.5)
-			(end -2.85 -2.499999)
-			(stroke
-				(width 0.05)
-				(type solid)
-			)
-			(layer "F.CrtYd")
-		)
-		(fp_line
-			(start -2.85 -2.499999)
-			(end 2.850001 -2.5)
-			(stroke
-				(width 0.05)
-				(type solid)
-			)
-			(layer "F.CrtYd")
-		)
 		(fp_text user "${REFERENCE}"
-			(at 0 0 45)
+			(at 0 0 90)
 			(layer "F.Fab")
 			(effects
@@
 		)
 		(pad "1" smd rect
-			(at -2.580001 0 225)
+			(at -2.580001 0 270)
 			(size 2.01 5.4)
 			(layers "F.Cu" "F.Mask" "F.Paste")
@@
 		)
 		(pad "2" smd rect
-			(at 2.580001 0 225)
+			(at 2.580001 0 270)
 			(size 2.01 5.4)
 			(layers "F.Cu" "F.Mask" "F.Paste")
@@
 	)
 	(segment
-		(start 141.251186 42.848814)
-		(end 149 35.1)
+		(start 149 35.1)
+		(end 142.189998 41.910002)
 		(width 2)
 		(layer "F.Cu")
@@
 	)
 	(segment
-		(start 141.251186 42.848814)
-		(end 137.235176 42.848814)
+		(start 142.189998 41.910002)
+		(end 139.25 41.910002)
 		(width 2)
 		(layer "F.Cu")

Commit message: flsh
Parts:
- moved TP1 17.8 mm to (134.0, 44.5)
- moved TP3 15.0 mm to (138.5, 62.0)
- moved C3 2.17 mm to (135.8, 48.6)
Connections:
- TP3 pad 1: GND -> (no net)
Routing:
- net VIN: track 12.6 -> 0.00 mm
- net GND: track 0.00 -> 10.9 mm, vias 15 -> 14
- net Net-(U2-FB): track 12.9 -> 15.6 mm, vias 2 -> 0

Commit message: zener
Parts:
- added DZ1: ZENER, easyeda2kicad:SOD-123FL_L2.6-W1.6-LS3.5-RD, F.Cu at (152.4, 64.2)
- added R1: 2kΩ, easyeda2kicad:R1206, F.Cu at (146.5, 66.4)
- moved TP5_EN1 4.00 mm to (157.8, 64.8)
- moved RS1 0.92 mm to (146.7, 63.4)
- moved TP3 0.06 mm to (138.5, 62.0)
Connections:
- RS1 pad 1: Net-(U2-FB) -> Net-(R1-Pad2)
- TP3 pad 1: (no net) -> GND
- U2 pad 5: Net-(U2-FB) -> Net-(DZ1-A)
Routing:
- net Net-(DZ1-A): track 0.00 -> 23.0 mm
- net Net-(U2-FB): track 15.6 -> 0.00 mm
- net VOUT: track 18.8 -> 32.8 mm
- net Net-(U2-EN): track 22.0 -> 31.2 mm
- net Net-(R1-Pad2): track 0.00 -> 3.65 mm
- net GND: vias 14 -> 16

Commit message: incremental small + cosmetic changes
It looks so pretty now
I also know that I'm distracting myself and I should do something else now
Parts:
- added H1: MountingHole, MountingHole:MountingHole_3.2mm_M3, F.Cu at (165.9, 48.6)
- C1: footprint easyeda2kicad:C2220 -> Capacitor_SMD:C_2220_5750Metric
- C3, C4: footprint easyeda2kicad:C1206 -> Capacitor_SMD:C_1206_3216Metric
- DZ1: footprint easyeda2kicad:SOD-123FL_L2.6-W1.6-LS3.5-RD -> Diode_SMD:D_SOD-123F
- R1: footprint easyeda2kicad:R1206 -> Resistor_SMD:R_1206_3216Metric
- moved TP2 4.20 mm to (165.5, 42.3)
- moved TP4 1.81 mm to (166.4, 54.8)
- moved TP5_EN1 0.87 mm to (157.0, 65.0)
- moved C1 0.23 mm to (139.4, 39.5)
Connections:
- net VOUT renamed LED+
- R1 pad 2: Net-(R1-Pad2) -> LED-
- RS1 pad 1: Net-(R1-Pad2) -> GND
- RS1 pad 2: GND -> LED-
- TP4 pad 1: GND -> LED-
Routing:
- net LED-: track 0.00 -> 35.6 mm
- net Net-(R1-Pad2): track 3.65 -> 0.00 mm
- net LED+: track 32.8 -> 31.3 mm
- net Net-(DZ1-A): track 23.0 -> 22.0 mm
- net GND: track 10.9 -> 10.8 mm, vias 16 -> 14
Other:
- board text added: "LED+"
- board text added: "LED-"
- board text removed: "VOUT"

Commit message: idk
Parts:
- D1: footprint easyeda2kicad:SMA_L4.4-W2.8-LS5.4-RD -> Diode_SMD:D_SMA
- RS1: footprint easyeda2kicad:RES-SMD_L6.4-W3.2-R2512 -> Resistor_SMD:R_2512_6332Metric
- moved RS1 1.28 mm to (145.4, 63.4)
- moved D1 0.72 mm to (157.4, 44.2)
- moved R1 0.24 mm to (146.3, 66.4)
Routing:
- net LED-: track 35.6 -> 38.4 mm
- net Net-(DZ1-A): track 22.0 -> 20.4 mm
- net LED+: track 31.3 -> 30.6 mm
- net GND: vias 14 -> 13
