File: PCB/flsh/flsh.kicad_sch (KiCad schematic)
At the start: 10 parts, among them U1 0.18Ω, U2 0.18Ω, U3 0.18Ω, U4 0.18Ω, U5 0.18Ω

Commit message: flsh!!
Parts:
- removed U1, U2, U3, U4, U5: 0.18Ω, easyeda2kicad:R1206, symbol lcsc:HOLRT1206-1W-180MR-1%
- added C1, C2, C3, C4, C5, C6, C7, C8: C_US, Capacitor_SMD:C_1206_3216Metric, symbol Device:C_US
- added LED6, LED7, LED8, LED9: GW PUSTA1.PM-PBQB-XX52-1-1050-R18, easyeda2kicad:LED-SMD_3P-L3.7-W3.7_GW-PUSTA1.PM-NAPD-XX510-1-1050-R18, symbol lcsc:GWPUSTA1.PM-PBQB-XX52-1-1050-R18
- added TP1, TP2: TestPoint, TestPoint:TestPoint_Pad_D1.0mm, symbol Connector:TestPoint
Connections:
- net GND: now also C4.1, LED9.2 (C), LED9.3 (C), TP2.1; no longer LED1.2 (C), LED1.3 (C), LED2.2 (C), LED2.3 (C), LED3.2 (C), LED3.3 (C), LED4.2 (C), LED4.3 (C), LED5.2 (C), LED5.3 (C)
- net LED_VCC: now also C1.2, LED6.1 (A), TP1.1
- net at LED5.1 (A): now also LED4.2 (C), LED4.3 (C), C3.2, C7.1
- net at LED2.1 (A): now also LED1.2 (C), LED1.3 (C), C2.1, C6.2
- net at LED1.1 (A): now also C2.2, C5.1, LED7.2 (C), LED7.3 (C)
- net at LED3.1 (A): now also LED2.2 (C), LED2.3 (C), C6.1
- net at LED4.1 (A): now also LED3.2 (C), LED3.3 (C), C7.2
- new net: C1.1, C5.2, LED6.2 (C), LED6.3 (C), LED7.1 (A)
- new net: C3.1, C8.2, LED5.2 (C), LED5.3 (C), LED8.1 (A)
- new net: C4.2, C8.1, LED8.2 (C), LED8.3 (C), LED9.1 (A)

Commit message: operation copy TI step 1
Parts:
- removed C1, C2, C3, C4, C5, C6, C7, C8: C_US, Capacitor_SMD:C_1206_3216Metric, symbol Device:C_US
- removed LED1, LED2, LED3, LED4, LED5, LED6, LED7, LED8, LED9: GW PUSTA1.PM-PBQB-XX52-1-1050-R18, easyeda2kicad:LED-SMD_3P-L3.7-W3.7_GW-PUSTA1.PM-NAPD-XX510-1-1050-R18, symbol lcsc:GWPUSTA1.PM-PBQB-XX52-1-1050-R18
- removed TP1, TP2: TestPoint, TestPoint:TestPoint_Pad_D1.0mm, symbol Connector:TestPoint
- added CComp: 150nF 16V, easyeda2kicad:C0805, symbol lcsc:CC0805KRX7R9BB154
- added CComp2: 8.2nF 50V X7R, easyeda2kicad:C0805, symbol lcsc:CC0805JRX7R9BB822
- added CFILT: 10pF, easyeda2kicad:C0805, symbol lcsc:CC0805JRNPO9BN100
- added CIN, CIN2: UUD1E471MNL1GS, easyeda2kicad:CAP-SMD_BD10.0-L10.3-W10.3-LS11.0-FD, symbol lcsc:UUD1E471MNL1GS
- added Cbyp: 100nF 25V X7R 0805, easyeda2kicad:C0805, symbol lcsc:0805B104K250NT
- added Cout: EEHZA1H101P, easyeda2kicad:CAP-SMD_BD10.0-L10.3-W10.3-FD, symbol lcsc:EEHZA1H101P
- added D1: SS24FL, easyeda2kicad:SOD-123FL_L2.8-W1.8-LS3.6-RD, symbol lcsc:SS24FL_C894433
- added L1: XAL1010-562MED, easyeda2kicad:IND-SMD_L11.3-W10.0_XAL1010-332ME, symbol lcsc:XAL1010-562MED
- added M1: IAUCN04S7L028ATMA1, easyeda2kicad:TDSON-8_L6.0-W5.0-P1.27-LS6.2-BL_1, symbol lcsc:IAUCN04S7L028ATMA1
- added RCOMP: 2.21k, easyeda2kicad:R0805, symbol lcsc:AR05ATS2211
- added RFB1: 976Ω, easyeda2kicad:R0805, symbol lcsc:FRC0805F9760TS
- added RFB2: 12kΩ, easyeda2kicad:R0805, symbol lcsc:RT0805BRE0721KL
- added RFILT: 100Ω, easyeda2kicad:R0805, symbol lcsc:RC0805FR-07100RL
- added Rfadj1: 105kΩ, easyeda2kicad:R0805, symbol lcsc:FRC0805F1053TS
- added Rsense: 3mΩ 1W sense, easyeda2kicad:RES-SMD_L6.4-W3.2-A, symbol lcsc:FPM253WFR003TML
- added U1: LM3478MM, easyeda2kicad:VSSOP-8_L3.0-W3.0-P0.65-LS5.0-BL, symbol lcsc:LM3478MM
Connections:
- net GND: now also CComp2.1, CFILT.1, CIN.2, CIN2.2, Cbyp.1, Cout.2, RCOMP.1, RFB1.1, Rfadj1.2, Rsense.1, U1.4 (AGND), U1.5 (PGND)
- new net: RFB1.2, RFB2.1, U1.3 (FB)
- new net: D1.2 (A), L1.2, M1.5 (D)
- new net: Rfadj1.1, U1.7 (FA/SD)
- new net: M1.1 (S), RFILT.2, Rsense.2
- new net: CComp.1, RCOMP.2
- new net COMP: CComp.2, CComp2.2, U1.2 (COMP)
- new net DR: M1.4 (G), U1.6 (DR)
- new net IOUT: Cout.1, D1.1 (C), RFB2.2
- new net ISEN: CFILT.2, RFILT.1, U1.1 (ISEN)
- new net VIN: CIN.1, CIN2.1, Cbyp.2, L1.1, U1.8 (VIN)

Commit message: more layout
Parts:
- added TP1, TP2, TP3, TP4: TestPoint, TestPoint:TestPoint_Pad_D4.0mm, symbol Connector:TestPoint
- renumbered CComp to CComp1, CFILT to CFILT1, CIN to CIN1, Cbyp to Cbyp1, Cout to Cout1, RCOMP to RCOMP1, RFILT to RFILT1, Rsense to Rsense1
Connections:
- net GND: now also TP3.1, TP4.1
- net IOUT: now also TP2.1
- net VIN: now also TP1.1

Commit message: a
Parts:
- added Cout2: EEHZA1H101P, easyeda2kicad:CAP-SMD_BD10.0-L10.3-W10.3-FD, symbol lcsc:EEHZA1H101P
Connections:
- net GND: now also Cout2.2
- net IOUT: now also Cout2.1
Changed lines of the file:
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@@
+	)
+	(junction
+		(at 264.16 83.82)
+		(diameter 0)
+		(color 0 0 0 0)
 	)
 	(junction
@@
 	(wire
 		(pts
-			(xy 254 83.82) (xy 243.84 83.82)
+			(xy 271.78 83.82) (xy 264.16 83.82)
 		)
 		(stroke
@@
 		(pts
 			(xy 151.13 88.9) (xy 157.48 88.9)
+		)
+		(stroke
+			(width 0)
+			(type default)
+		)
+	)
+	(wire
+		(pts
+			(xy 264.16 83.82) (xy 243.84 83.82)
 		)
 		(stroke
@@
 	(global_label "IOUT"
 		(shape input)
-		(at 254 83.82 0)
+		(at 271.78 83.82 0)
 		(fields_autoplaced yes)
 		(effects
@@
 		)
 		(property "Intersheetrefs" "${INTERSHEET_REFS}"
-			(at 261.2186 83.82 0)
+			(at 278.9986 83.82 0)
 			(hide yes)
 			(show_name no)
@@
 	)
 	(symbol
+		(lib_id "lcsc:EEHZA1H101P")
+		(at 264.16 87.63 0)
+		(unit 1)
+		(body_style 1)
+		(exclude_from_sim no)
+		(in_bom yes)
+		(on_board yes)
+		(in_pos_files yes)
+		(dnp no)
+		(fields_autoplaced yes)
+		(property "Reference" "Cout2"
+			(at 267.97 85.7549 0)
+			(show_name no)
+			(do_not_autoplace no)
+			(effects
+				(font
+					(size 1.27 1.27)
+				)
+				(justify left)
+			)
+		)
+		(property "Value" "EEHZA1H101P"
+			(at 267.97 88.2949 0)
+			(show_name no)
+			(do_not_autoplace no)
+			(effects
+				(font
+					(size 1.27 1.27)
+				)
+				(justify left)
+			)
+		)
+		(property "Footprint" "easyeda2kicad:CAP-SMD_BD10.0-L10.3-W10.3-FD"
+			(at 264.16 99.06 0)
+			(hide yes)
+			(show_name no)
+			(do_not_autoplace no)
+			(effects
+				(font
+					(size 1.27 1.27)
+				)
+			)
+		)
+		(property "Datasheet" "https://lcsc.com/product-detail/Aluminum-Electrolytic-Capacitors-SMD_PANASONIC_EEHZA1H101P_100uF-101-20-50V_C109086.html"
+			(at 264.16 101.6 0)
+			(hide yes)
+			(show_name no)
+			(do_not_autoplace no)
+			(effects
+				(font
+					(size 1.27 1.27)
+				)
+			)
+		)
+		(property "Description" ""
+			(at 264.16 87.63 0)
+			(hide yes)
+			(show_name no)
+			(do_not_autoplace no)
+			(effects
+				(font
+					(size 1.27 1.27)
+				)
+			)
+		)
+		(property "Manufacturer" "PANASONIC(松下)"
+			(at 264.16 104.14 0)
+			(hide yes)
+			(show_name no)
+			(do_not_autoplace no)
+			(effects
+				(font
+					(size 1.27 1.27)
+				)
+			)
+		)
+		(property "MPN" "EEHZA1H101P"
+			(at 264.16 106.68 0)
+			(hide yes)
+			(show_name no)
+			(do_not_autoplace no)
+			(effects
+				(font
+					(size 1.27 1.27)
+				)
+			)
+		)
+		(property "LCSC Part" "C109086"
+			(at 264.16 109.22 0)
+			(hide yes)
+			(show_name no)
+			(do_not_autoplace no)
+			(effects
+				(font
+					(size 1.27 1.27)
+				)
+			)
+		)
+		(pin "1"
+		)
+		(pin "2"
+		)
+		(instances
+			(project "flsh"
+				(path "/08418876-6758-4030-87ef-cfeed83d90aa"
+					(reference "Cout2")
+					(unit 1)
+				)
+			)
+		)
+	)
+	(symbol
 		(lib_id "power:GND")
 		(at 90.17 90.17 0)
@@
 					(unit 1)
 				)
+			)
+		)
+	)
+	(symbol
+		(lib_id "power:GND")
+		(at 264.16 91.44 0)
+		(unit 1)
+		(body_style 1)
+		(exclude_from_sim no)
+		(in_bom yes)
+		(on_board yes)
+		(in_pos_files yes)
+		(dnp no)
+		(fields_autoplaced yes)
+		(property "Reference" "#PWR012"
+			(at 264.16 97.79 0)
+			(hide yes)
+			(show_name no)
+			(do_not_autoplace no)
+			(effects
+				(font
+					(size 1.27 1.27)
+				)
+			)
+		)
+		(property "Value" "GND"
+			(at 264.16 96.52 0)
+			(show_name no)
+			(do_not_autoplace no)
+			(effects
+				(font
+					(size 1.27 1.27)
+				)
+			)
+		)
+		(property "Footprint" ""
+			(at 264.16 91.44 0)
+			(hide yes)
+			(show_name no)
+			(do_not_autoplace no)
+			(effects
+				(font
+					(size 1.27 1.27)
+				)
+			)
+		)
+		(property "Datasheet" ""
+			(at 264.16 91.44 0)
+			(hide yes)
+			(show_name no)
+			(do_not_autoplace no)
+			(effects
+				(font
+					(size 1.27 1.27)
+				)
+			)
+		)
+		(property "Description" "Power symbol creates a global label with name \"GND\" , ground"
+			(at 264.16 91.44 0)
+			(hide yes)
+			(show_name no)
+			(do_not_autoplace no)
+			(effects
+				(font
+					(size 1.27 1.27)
+				)
+			)
+		)
+		(pin "1"
+		)
+		(instances
+			(project "flsh"
+				(path "/08418876-6758-4030-87ef-cfeed83d90aa"
+					(reference "#PWR012")
+					(unit 1)
+				)

Commit message: lwk redid the whole pcb
Parts:
- removed CComp1: 150nF 16V, easyeda2kicad:C0805, symbol lcsc:CC0805KRX7R9BB154
- removed CComp2: 8.2nF 50V X7R, easyeda2kicad:C0805, symbol lcsc:CC0805JRX7R9BB822
- removed CFILT1: 10pF, easyeda2kicad:C0805, symbol lcsc:CC0805JRNPO9BN100
- removed CIN1, CIN2: UUD1E471MNL1GS, easyeda2kicad:CAP-SMD_BD10.0-L10.3-W10.3-LS11.0-FD, symbol lcsc:UUD1E471MNL1GS
- removed Cbyp1: 100nF 25V X7R 0805, easyeda2kicad:C0805, symbol lcsc:0805B104K250NT
- removed Cout1, Cout2: EEHZA1H101P, easyeda2kicad:CAP-SMD_BD10.0-L10.3-W10.3-FD, symbol lcsc:EEHZA1H101P
- removed D1: SS24FL, easyeda2kicad:SOD-123FL_L2.8-W1.8-LS3.6-RD, symbol lcsc:SS24FL_C894433
- removed L1: XAL1010-562MED, easyeda2kicad:IND-SMD_L11.3-W10.0_XAL1010-332ME, symbol lcsc:XAL1010-562MED
- removed M1: IAUCN04S7L028ATMA1, easyeda2kicad:TDSON-8_L6.0-W5.0-P1.27-LS6.2-BL_1, symbol lcsc:IAUCN04S7L028ATMA1
- removed RCOMP1: 2.21k, easyeda2kicad:R0805, symbol lcsc:AR05ATS2211
- removed RFB1: 976Ω, easyeda2kicad:R0805, symbol lcsc:FRC0805F9760TS
- removed RFB2: 12kΩ, easyeda2kicad:R0805, symbol lcsc:RT0805BRE0721KL
- removed RFILT1: 100Ω, easyeda2kicad:R0805, symbol lcsc:RC0805FR-07100RL
- removed Rfadj1: 105kΩ, easyeda2kicad:R0805, symbol lcsc:FRC0805F1053TS
- removed Rsense1: 3mΩ 1W sense, easyeda2kicad:RES-SMD_L6.4-W3.2-A, symbol lcsc:FPM253WFR003TML
- removed U1: LM3478MM, easyeda2kicad:VSSOP-8_L3.0-W3.0-P0.65-LS5.0-BL, symbol lcsc:LM3478MM
- added C1: 47uF 35V, easyeda2kicad:C2220, symbol easyeda2kicad:CKG57NX7R1H476MT009W
- added C2: 100uF 63V, easyeda2kicad:CAP-SMD_BD10.0-L10.3-W10.3-FD, symbol easyeda2kicad:MA80V100M10X12
- added C3, C4: 1uF, easyeda2kicad:C1206, symbol easyeda2kicad:CL31B105KCHNNNE
- added D1: SS38_C64999, easyeda2kicad:SMA_L4.4-W2.8-LS5.4-RD, symbol easyeda2kicad:SS38_C64999
- added L1: YSPI1365-470M, easyeda2kicad:IND-SMD_L13.8-W12.6_H6.5, symbol easyeda2kicad:YSPI1365-470M
- added RS1: JER2512F2R220, easyeda2kicad:RES-SMD_L6.4-W3.2-R2512, symbol easyeda2kicad:JER2512F2R220
- added TP5_EN1: TestPoint, TestPoint:TestPoint_Pad_D4.0mm, symbol Connector:TestPoint
- added U2: XL6006E1, easyeda2kicad:TO-263-5_L10.2-W9.9-P1.70-LS14.4-TL, symbol easyeda2kicad:XL6006E1
Connections:
- net GND: now also C1.1, C2.2, C3.1, C4.1, RS1.2, U2.1 (GND)
- net VIN: now also C1.2, C3.2, L1.1, U2.4 (VIN)
- net IOUT renamed VOUT
- net VOUT: now also C2.1, C4.2, D1.1 (K)
- new net: TP5_EN1.1, U2.2 (EN)
- new net: D1.2 (A), L1.2, U2.3 (SW), U2.6 (SW)
- new net: RS1.1, U2.5 (FB)

Commit message: zener
Parts:
- added DZ1: ZENER, easyeda2kicad:SOD-123FL_L2.6-W1.6-LS3.5-RD, symbol easyeda2kicad:BZT52C39WT
- added R1: 2kΩ, easyeda2kicad:R1206, symbol easyeda2kicad:RC1206FR-072KL
Connections:
- net VOUT: now also DZ1.1 (K)
- net at U2.5 (FB): now also DZ1.2 (A), R1.1; no longer RS1.1
- new net: R1.2, RS1.1
Other:
- moved on the sheet: RS1

Commit message: incremental small + cosmetic changes
It looks so pretty now
I also know that I'm distracting myself and I should do something else now
Parts:
- added H1: MountingHole, MountingHole:MountingHole_3.2mm_M3, symbol Mechanical:MountingHole
- C1: footprint easyeda2kicad:C2220 -> Capacitor_SMD:C_2220_5750Metric; LCSC Part C49297048 -> C27840590; MPN CKG57NX7R1H476MT009W -> KTJ350B476M55BFT00; Manufacturer TDK -> NCC
- C3, C4: footprint easyeda2kicad:C1206 -> Capacitor_SMD:C_1206_3216Metric
- DZ1: footprint easyeda2kicad:SOD-123FL_L2.6-W1.6-LS3.5-RD -> Diode_SMD:D_SOD-123F
- R1: footprint easyeda2kicad:R1206 -> Resistor_SMD:R_1206_3216Metric
Connections:
- net GND: now also RS1.1; no longer RS1.2, TP4.1
- net LED-: now reaches R1.2
- net LED-: now also RS1.2, TP4.1; no longer RS1.1
- net VOUT renamed LED+
Other:
- moved on the sheet: C1, C3, D1, DZ1, L1, RS1, TP1

Commit message: idk
Parts:
- D1: footprint easyeda2kicad:SMA_L4.4-W2.8-LS5.4-RD -> Diode_SMD:D_SMA
- RS1: footprint easyeda2kicad:RES-SMD_L6.4-W3.2-R2512 -> Resistor_SMD:R_2512_6332Metric
Changed lines of the file:
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@@
 			)
 		)
-		(property "Footprint" "easyeda2kicad:RES-SMD_L6.4-W3.2-R2512"
+		(property "Footprint" "Resistor_SMD:R_2512_6332Metric"
 			(at 158.75 101.6 0)
 			(hide yes)
@@
 			)
 		)
-		(property "Footprint" "easyeda2kicad:SMA_L4.4-W2.8-LS5.4-RD"
+		(property "Footprint" "Diode_SMD:D_SMA"
 			(at 109.22 57.15 0)
 			(hide yes)
