File: PCB/flsh/flsh_batt.kicad_sch (KiCad schematic)
At the start: 5 parts

Commit message: flsh batt!
Parts:
- removed BT1, BT2: Battery_Cell, symbol Device:Battery_Cell
- added BT1, BT2: 1121, flsh_batt:BAT_1121, symbol flsh_batt:1121
Connections:
- net GND: now also BT2.N
- net VCC: now also BT1.P
- net at TP3.1: now also BT1.N, BT2.P
Other:
- moved on the sheet: TP1, TP2
